File: Henning/Henning.sch (KiCad schematic (older format))
At the start: 16 parts

Commit message: Design by prof dr Peter A Henning
Parts:
- removed D?: 1N4148, symbol Diode_Bridge
- added D1, D2, D3, D4: D, Diodes_ThroughHole:Diode_DO-35_SOD27_Horizontal_RM10, symbol D
- added P1: RS232, Socket_Strips:Socket_Strip_Angled_1x04, symbol CONN_01X04
- added P2: EBUS, Terminal_Blocks:TerminalBlock_WAGO-236_2Stift_RM5mm_2pol, symbol CONN_01X02
- C1: renamed from C?; footprint (none) -> Capacitors_ThroughHole:C_Radial_D5_L6_P2.5
- D5: renamed from D?; footprint (none) -> Diodes_ThroughHole:Diode_DO-35_SOD27_Horizontal_RM10
- Q1: renamed from Q?; footprint (none) -> TO_SOT_Packages_THT:TO-220_Neutral123_Horizontal
- R1, R2, R3, R4, R5: renamed from R?; footprint (none) -> Resistors_ThroughHole:Resistor_Horizontal_RM10mm
- RV1: renamed from RV?; footprint (none) -> Potentiometers:Potentiometer_Bourns_3296W_3-8Zoll_Inline_ScrewUp
- U1: renamed from U?; footprint (none) -> Housings_DIP:DIP-14_W7.62mm
- U2, U4: renamed from U?; footprint (none) -> Housings_DIP:DIP-6_W7.62mm
- U3: renamed from U?; footprint (none) -> TO_SOT_Packages_THT:TO-92_Molded_Wide
Connections:
- net EBUS1: now also D1.2 (A), D2.1 (K), P2.2 (P2)
- net EBUS2: now also D3.1 (K), D4.2 (A), P2.1 (P1)
- net GND: now also P1.1 (P1)
- net RXD: now also P1.3 (P3)
- net TXD: now also U1.1, U1.2, P1.2 (P2); no longer U1.8, U1.9
- net VDD: now also U1.9, P1.4 (P4); no longer U1.2
- net at Q1.1, U4.2: now also D1.1 (K), D4.1 (K); no longer C1.2, U3.2 (GND)
- net at D5.1 (K), R5.1, U3.1 (VI): now also D2.2 (A), D3.2 (A)
- net at R2.2: now also U1.3; no longer U1.10
- net at R3.1, U4.4: now also U1.8; no longer U1.1
- net at U1.5: now also U1.10; no longer U1.3
Changed lines of the file:
@@
 Comment4 ""
 $EndDescr
-$Comp
-L Diode_Bridge D?
-U 1 1 57E43393
-P 8700 2900
-F 0 "D?" H 8450 3200 50  0000 C CNN
-F 1 "1N4148" H 9050 2550 50  0000 C CNN
-F 2 "" H 8700 2900 50  0000 C CNN
-F 3 "" H 8700 2900 50  0000 C CNN
-	1    8700 2900
-	1    0    0    -1
-$EndComp
 Text GLabel 9700 2300 2    60   Input ~ 0
 EBUS1
-Text GLabel 9700 3500 2    60   Input ~ 0
+Text GLabel 9700 2700 2    60   Input ~ 0
 EBUS2
-Wire Wire Line
-	8700 2500 8700 2300
-Wire Wire Line
-	8700 2300 9700 2300
-Wire Wire Line
-	9700 3500 8700 3500
-Wire Wire Line
-	8700 3500 8700 3300
-$Comp
-L ZENER D?
+$Comp
+L ZENER D5
 U 1 1 57E433F4
 P 9100 3800
-F 0 "D?" H 9100 3900 50  0000 C CNN
+F 0 "D5" H 9100 3900 50  0000 C CNN
 F 1 "ZPY7.5V 1.3W" H 9100 3700 50  0000 C CNN
-F 2 "" H 9100 3800 50  0000 C CNN
+F 2 "Diodes_ThroughHole:Diode_DO-35_SOD27_Horizontal_RM10" H 9100 3800 50  0001 C CNN
 F 3 "" H 9100 3800 50  0000 C CNN
 	1    9100 3800
@@
 $EndComp
 $Comp
-L R R?
+L R R4
 U 1 1 57E434B6
 P 7250 3500
-F 0 "R?" V 7330 3500 50  0000 C CNN
+F 0 "R4" V 7330 3500 50  0000 C CNN
 F 1 "22k" V 7250 3500 50  0000 C CNN
-F 2 "" V 7180 3500 50  0000 C CNN
+F 2 "Resistors_ThroughHole:Resistor_Horizontal_RM10mm" V 7180 3500 50  0001 C CNN
 F 3 "" H 7250 3500 50  0000 C CNN
 	1    7250 3500
@@
 $EndComp
 $Comp
-L R R?
+L R R5
 U 1 1 57E434EC
 P 8800 1350
-F 0 "R?" V 8880 1350 50  0000 C CNN
+F 0 "R5" V 8880 1350 50  0000 C CNN
 F 1 "3k3" V 8800 1350 50  0000 C CNN
-F 2 "" V 8730 1350 50  0000 C CNN
+F 2 "Resistors_ThroughHole:Resistor_Horizontal_RM10mm" V 8730 1350 50  0001 C CNN
 F 3 "" H 8800 1350 50  0000 C CNN
 	1    8800 1350
@@
 $EndComp
 $Comp
-L 78L05 U?
+L 78L05 U3
 U 1 1 57E4352D
 P 6800 3950
-F 0 "U?" H 6950 3754 50  0000 C CNN
+F 0 "U3" H 6950 3754 50  0000 C CNN
 F 1 "78L05" H 6800 4150 50  0000 C CNN
-F 2 "" H 6800 3950 50  0000 C CNN
+F 2 "TO_SOT_Packages_THT:TO-92_Molded_Wide" H 6800 3950 50  0001 C CNN
 F 3 "" H 6800 3950 50  0000 C CNN
 	1    6800 3950
@@
 $EndComp
 $Comp
-L Darl_NPN Q?
+L Darl_NPN Q1
 U 1 1 57E43564
 P 7900 3500
-F 0 "Q?" H 7900 3700 50  0000 C CNN
+F 0 "Q1" H 7900 3700 50  0000 C CNN
 F 1 "BD645" H 7700 3350 50  0000 C CNN
-F 2 "" H 7900 3450 50  0000 C CNN
+F 2 "TO_SOT_Packages_THT:TO-220_Neutral123_Horizontal" H 7900 3450 50  0001 C CNN
 F 3 "" H 7900 3450 50  0000 C CNN
 	1    7900 3500
@@
 $EndComp
 $Comp
-L CP C?
+L CP C1
 U 1 1 57E435D0
 P 6200 3550
-F 0 "C?" H 6225 3650 50  0000 L CNN
+F 0 "C1" H 6225 3650 50  0000 L CNN
 F 1 "CP" H 6225 3450 50  0000 L CNN
-F 2 "" H 6238 3400 50  0000 C CNN
+F 2 "Capacitors_ThroughHole:C_Radial_D5_L6_P2.5" H 6238 3400 50  0001 C CNN
 F 3 "" H 6200 3550 50  0000 C CNN
 	1    6200 3550
@@
 $EndComp
 $Comp
-L R R?
+L R R2
 U 1 1 57E43613
 P 4650 4600
-F 0 "R?" V 4730 4600 50  0000 C CNN
+F 0 "R2" V 4730 4600 50  0000 C CNN
 F 1 "470" V 4650 4600 50  0000 C CNN
-F 2 "" V 4580 4600 50  0000 C CNN
+F 2 "Resistors_ThroughHole:Resistor_Horizontal_RM10mm" V 4580 4600 50  0001 C CNN
 F 3 "" H 4650 4600 50  0000 C CNN
 	1    4650 4600
@@
 $EndComp
 $Comp
-L R R?
+L R R3
 U 1 1 57E43651
 P 5450 2800
-F 0 "R?" V 5530 2800 50  0000 C CNN
+F 0 "R3" V 5530 2800 50  0000 C CNN
 F 1 "1k" V 5450 2800 50  0000 C CNN
-F 2 "" V 5380 2800 50  0000 C CNN
+F 2 "Resistors_ThroughHole:Resistor_Horizontal_RM10mm" V 5380 2800 50  0001 C CNN
 F 3 "" H 5450 2800 50  0000 C CNN
 	1    5450 2800
@@
 $EndComp
 $Comp
-L R R?
+L R R1
 U 1 1 57E4369F
 P 4050 1650
-F 0 "R?" V 4130 1650 50  0000 C CNN
+F 0 "R1" V 4130 1650 50  0000 C CNN
 F 1 "10k" V 4050 1650 50  0000 C CNN
-F 2 "" V 3980 1650 50  0000 C CNN
+F 2 "Resistors_ThroughHole:Resistor_Horizontal_RM10mm" V 3980 1650 50  0001 C CNN
 F 3 "" H 4050 1650 50  0000 C CNN
 	1    4050 1650
@@
 $EndComp
 $Comp
-L POT RV?
+L POT RV1
 U 1 1 57E43705
 P 4850 2800
-F 0 "RV?" H 4850 2720 50  0000 C CNN
+F 0 "RV1" H 4850 2720 50  0000 C CNN
 F 1 "20k" H 4850 2800 50  0000 C CNN
-F 2 "" H 4850 2800 50  0000 C CNN
+F 2 "Potentiometers:Potentiometer_Bourns_3296W_3-8Zoll_Inline_ScrewUp" H 4850 2800 50  0001 C CNN
 F 3 "" H 4850 2800 50  0000 C CNN
 	1    4850 2800
@@
 $EndComp
 $Comp
-L 4011 U?
-U 1 1 57E43757
+L 4011 U1
+U 3 1 57E43757
 P 6200 1700
-F 0 "U?" H 6200 1750 50  0000 C CNN
+F 0 "U1" H 6200 1750 50  0000 C CNN
 F 1 "4011" H 6200 1650 50  0000 C CNN
-F 2 "" H 6200 1700 60  0000 C CNN
+F 2 "Housings_DIP:DIP-14_W7.62mm" H 6200 1700 60  0001 C CNN
 F 3 "" H 6200 1700 60  0000 C CNN
-	1    6200 1700
-	-1   0    0    1
-$EndComp
-$Comp
-L CNY17-1 U?
+	3    6200 1700
+	-1   0    0    1
+$EndComp
+$Comp
+L CNY17-1 U4
 U 1 1 57E43851
 P 7800 1450
-F 0 "U?" H 7600 1650 50  0000 L CNN
+F 0 "U4" H 7600 1650 50  0000 L CNN
 F 1 "CNY17-1" H 7800 1650 50  0000 L CNN
-F 2 "" H 7800 1450 50  0000 L CNN
+F 2 "Housings_DIP:DIP-6_W7.62mm" H 7800 1450 50  0001 L CNN
 F 3 "" H 7800 1450 50  0000 L CNN
 	1    7800 1450
@@
 $EndComp
 $Comp
-L CNY17-1 U?
+L CNY17-1 U2
 U 1 1 57E438AA
 P 5400 4000
-F 0 "U?" H 5200 4200 50  0000 L CNN
+F 0 "U2" H 5200 4200 50  0000 L CNN
 F 1 "CNY17-1" H 5400 4200 50  0000 L CNN
-F 2 "" H 5400 4000 50  0000 L CNN
+F 2 "Housings_DIP:DIP-6_W7.62mm" H 5400 4000 50  0001 L CNN
 F 3 "" H 5400 4000 50  0000 L CNN
 	1    5400 4000
@@
 Wire Wire Line
 	9400 3800 9300 3800
-Wire Wire Line
-	9100 2900 9400 2900
-Connection ~ 9400 2900
-Wire Wire Line
-	6200 2900 8300 2900
 Connection ~ 8200 2900
 Wire Wire Line
@@
 	3900 1250 7100 1250
 $Comp
-L 4011 U?
+L 4011 U1
 U 2 1 57E4437E
 P 4800 1600
-F 0 "U?" H 4800 1650 50  0000 C CNN
+F 0 "U1" H 4800 1650 50  0000 C CNN
 F 1 "4011" H 4800 1550 50  0000 C CNN
-F 2 "" H 4800 1600 60  0000 C CNN
+F 2 "Housings_DIP:DIP-14_W7.62mm" H 4800 1600 60  0001 C CNN
 F 3 "" H 4800 1600 60  0000 C CNN
 	2    4800 1600
@@
 Connection ~ 4200 2100
 $Comp
-L 4011 U?
-U 3 1 57E44779
+L 4011 U1
+U 1 1 57E44779
 P 4200 3800
-F 0 "U?" H 4200 3850 50  0000 C CNN
+F 0 "U1" H 4200 3850 50  0000 C CNN
 F 1 "4011" H 4200 3750 50  0000 C CNN
-F 2 "" H 4200 3800 60  0000 C CNN
+F 2 "Housings_DIP:DIP-14_W7.62mm" H 4200 3800 60  0001 C CNN
 F 3 "" H 4200 3800 60  0000 C CNN
-	3    4200 3800
+	1    4200 3800
 	0    1    1    0
 $EndComp
@@
 Wire Wire Line
 	8200 1550 8200 3200
+$Comp
+L D D1
+U 1 1 57E456DB
+P 8750 2200
+F 0 "D1" H 8750 2300 50  0000 C CNN
+F 1 "D" H 8750 2100 50  0000 C CNN
+F 2 "Diodes_ThroughHole:Diode_DO-35_SOD27_Horizontal_RM10" H 8750 2200 50  0001 C CNN
+F 3 "" H 8750 2200 50  0000 C CNN
+	1    8750 2200
+	1    0    0    -1
+$EndComp
+$Comp
+L D D2
+U 1 1 57E45729
+P 8750 2400
+F 0 "D2" H 8750 2500 50  0000 C CNN
+F 1 "D" H 8750 2300 50  0000 C CNN
+F 2 "Diodes_ThroughHole:Diode_DO-35_SOD27_Horizontal_RM10" H 8750 2400 50  0001 C CNN
+F 3 "" H 8750 2400 50  0000 C CNN
+	1    8750 2400
+	-1   0    0    1
+$EndComp
+$Comp
+L D D3
+U 1 1 57E45775
+P 8750 2600
+F 0 "D3" H 8750 2700 50  0000 C CNN
+F 1 "D" H 8750 2500 50  0000 C CNN
+F 2 "Diodes_ThroughHole:Diode_DO-35_SOD27_Horizontal_RM10" H 8750 2600 50  0001 C CNN
+F 3 "" H 8750 2600 50  0000 C CNN
+	1    8750 2600
+	-1   0    0    1
+$EndComp
+$Comp
+L D D4
+U 1 1 57E457DF
+P 8750 2800
+F 0 "D4" H 8750 2900 50  0000 C CNN
+F 1 "D" H 8750 2700 50  0000 C CNN
+F 2 "Diodes_ThroughHole:Diode_DO-35_SOD27_Horizontal_RM10" H 8750 2800 50  0001 C CNN
+F 3 "" H 8750 2800 50  0000 C CNN
+	1    8750 2800
+	1    0    0    -1
+$EndComp
+Wire Wire Line
+	8900 2200 9000 2200
+Wire Wire Line
+	9000 2200 9000 2400
+Wire Wire Line
+	9000 2400 8900 2400
+Wire Wire Line
+	8900 2600 9000 2600
+Wire Wire Line
+	9000 2600 9000 2800
+Wire Wire Line
+	9000 2800 8900 2800
+Wire Wire Line
+	9700 2300 9000 2300
+Connection ~ 9000 2300
+Wire Wire Line
+	8600 2200 8500 2200
+Wire Wire Line
+	8500 2200 8500 2800
+Wire Wire Line
+	8500 2800 8600 2800
+Wire Wire Line
+	8600 2400 8600 2600
+Wire Wire Line
+	9400 2500 8600 2500
+Connection ~ 8600 2500
+Connection ~ 9400 2500
+Wire Wire Line
+	8500 2500 8200 2500
+Connection ~ 8200 2500
+Connection ~ 8500 2500
+Wire Wire Line
+	9000 2700 9700 2700
+Connection ~ 9000 2700
+$Comp
+L CONN_01X02 P2
+U 1 1 57E45DDB
+P 9200 5250
+F 0 "P2" H 9200 5400 50  0000 C CNN
+F 1 "EBUS" V 9300 5250 50  0000 C CNN
+F 2 "Terminal_Blocks:TerminalBlock_WAGO-236_2Stift_RM5mm_2pol" H 9200 5250 50  0001 C CNN
+F 3 "" H 9200 5250 50  0000 C CNN
+	1    9200 5250
+	-1   0    0    1
+$EndComp
+$Comp
+L CONN_01X04 P1
+U 1 1 57E45F11
+P 1900 2750
+F 0 "P1" H 1900 3000 50  0000 C CNN
+F 1 "RS232" V 2000 2750 50  0000 C CNN
+F 2 "Socket_Strips:Socket_Strip_Angled_1x04" H 1900 2750 50  0001 C CNN
+F 3 "" H 1900 2750 50  0000 C CNN
+	1    1900 2750
+	-1   0    0    1
+$EndComp
+Text GLabel 9800 5200 2    60   Input ~ 0
+EBUS1
+Text GLabel 10200 5300 2    60   Input ~ 0
+EBUS2
+Wire Wire Line
+	9800 5200 9400 5200
+Wire Wire Line
+	9400 5300 10200 5300
+Text GLabel 2300 2600 2    60   Input ~ 0
+VDD
+Text GLabel 2600 2700 2    60   Input ~ 0
+RXD
+Text GLabel 2300 2800 2    60   Input ~ 0
+TXD
+Text GLabel 2600 2900 2    60   Input ~ 0
+GND
+Wire Wire Line
+	2300 2600 2100 2600
+Wire Wire Line
+	2100 2700 2600 2700
+Wire Wire Line
+	2300 2800 2100 2800
+Wire Wire Line
+	2100 2900 2600 2900
 $EndSCHEMATC

Commit message: PCB generated, but with some errors.
Parts:
- P1: footprint Socket_Strips:Socket_Strip_Angled_1x04 -> Pin_Headers:Pin_Header_Straight_1x04
- Q1: footprint TO_SOT_Packages_THT:TO-220_Neutral123_Horizontal -> TO_SOT_Packages_THT:TO-220_Neutral123_Vertical
Connections:
- net GND is gone; now on net VSS: P1.1 (P1), RV1.2, RV1.3, U2.2
- net at U3.2 (GND): now also C1.2, D1.1 (K), D4.1 (K), Q1.1, U4.2
Changed lines of the file:
@@
 LIBS:contrib
 LIBS:valves
+LIBS:Henning-cache
 EELAYER 25 0
 EELAYER END
@@
 F 0 "Q1" H 7900 3700 50  0000 C CNN
 F 1 "BD645" H 7700 3350 50  0000 C CNN
-F 2 "TO_SOT_Packages_THT:TO-220_Neutral123_Horizontal" H 7900 3450 50  0001 C CNN
+F 2 "TO_SOT_Packages_THT:TO-220_Neutral123_Vertical" H 7900 3450 50  0001 C CNN
 F 3 "" H 7900 3450 50  0000 C CNN
 	1    7900 3500
@@
 	9400 4000 7200 4000
 Connection ~ 9400 3800
-Wire Wire Line
-	6800 3700 6800 2900
-Wire Wire Line
-	6200 3400 6200 2900
 Connection ~ 6800 2900
 Wire Wire Line
@@
 GND
 Wire Wire Line
-	3700 2400 3900 2400
+	3700 2400 5000 2400
 Wire Wire Line
 	3900 2400 3900 1250
@@
 F 0 "P1" H 1900 3000 50  0000 C CNN
 F 1 "RS232" V 2000 2750 50  0000 C CNN
-F 2 "Socket_Strips:Socket_Strip_Angled_1x04" H 1900 2750 50  0001 C CNN
+F 2 "Pin_Headers:Pin_Header_Straight_1x04" H 1900 2750 50  0001 C CNN
 F 3 "" H 1900 2750 50  0000 C CNN
 	1    1900 2750
@@
 Wire Wire Line
 	2100 2900 2600 2900
+Wire Wire Line
+	6800 3700 6800 2900
+Wire Wire Line
+	6200 2900 8200 2900
+Wire Wire Line
+	6200 2900 6200 3400
+Wire Wire Line
+	5000 1400 5000 800
+Wire Wire Line
+	5000 800  4300 800
+Wire Wire Line
+	4300 800  4300 2800
+Connection ~ 4300 2800
+Wire Wire Line
+	5000 2400 5000 1800
+Connection ~ 3900 2400
 $EndSCHEMATC

Commit message: Fixed PCB
Parts:
- D1, D2, D3, D4: value D -> 1N4148
Connections:
- net EBUS1: now also D1.1 (K), D2.2 (A); no longer D1.2 (A), D2.1 (K)
- net EBUS2: now also D3.2 (A), D4.1 (K); no longer D3.1 (K), D4.2 (A)
- net at D5.1 (K), R5.1, U3.1 (VI): now also D2.1 (K), D3.1 (K); no longer D2.2 (A), D3.2 (A)
- net at C1.2, Q1.1, U3.2 (GND)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: now also D1.2 (A), D4.2 (A); no longer D1.1 (K), D4.1 (K)
Changed lines of the file:
@@
 U 1 1 57E456DB
 P 8750 2200
-F 0 "D1" H 8750 2300 50  0000 C CNN
-F 1 "D" H 8750 2100 50  0000 C CNN
+F 0 "D1" H 8850 2300 50  0000 C CNN
+F 1 "1N4148" H 8600 2300 50  0000 C CNN
 F 2 "Diodes_ThroughHole:Diode_DO-35_SOD27_Horizontal_RM10" H 8750 2200 50  0001 C CNN
 F 3 "" H 8750 2200 50  0000 C CNN
 	1    8750 2200
-	1    0    0    -1
+	-1   0    0    -1
 $EndComp
 $Comp
@@
 U 1 1 57E45729
 P 8750 2400
-F 0 "D2" H 8750 2500 50  0000 C CNN
-F 1 "D" H 8750 2300 50  0000 C CNN
+F 0 "D2" H 8650 2300 50  0000 C CNN
+F 1 "1N4148" H 8900 2300 50  0000 C CNN
 F 2 "Diodes_ThroughHole:Diode_DO-35_SOD27_Horizontal_RM10" H 8750 2400 50  0001 C CNN
 F 3 "" H 8750 2400 50  0000 C CNN
 	1    8750 2400
-	-1   0    0    1
+	1    0    0    1
 $EndComp
 $Comp
@@
 U 1 1 57E45775
 P 8750 2600
-F 0 "D3" H 8750 2700 50  0000 C CNN
-F 1 "D" H 8750 2500 50  0000 C CNN
+F 0 "D3" H 8650 2500 50  0000 C CNN
+F 1 "1N4148" H 8900 2500 50  0000 C CNN
 F 2 "Diodes_ThroughHole:Diode_DO-35_SOD27_Horizontal_RM10" H 8750 2600 50  0001 C CNN
 F 3 "" H 8750 2600 50  0000 C CNN
 	1    8750 2600
-	-1   0    0    1
+	1    0    0    1
 $EndComp
 $Comp
@@
 U 1 1 57E457DF
 P 8750 2800
-F 0 "D4" H 8750 2900 50  0000 C CNN
-F 1 "D" H 8750 2700 50  0000 C CNN
+F 0 "D4" H 8850 2900 50  0000 C CNN
+F 1 "1N4148" H 8600 2900 50  0000 C CNN
 F 2 "Diodes_ThroughHole:Diode_DO-35_SOD27_Horizontal_RM10" H 8750 2800 50  0001 C CNN
 F 3 "" H 8750 2800 50  0000 C CNN
 	1    8750 2800
-	1    0    0    -1
+	-1   0    0    -1
 $EndComp
 Wire Wire Line
