File: Peter_A_Henning/Henning.kicad_pcb (KiCad board)
At the start: 2 copper layers, 68 x 38 mm, 19 parts, among them P1 RS232, P2 EBUS, Q1 BD645, U1 4011, U2 CNY17-1, U3 78L05, U4 CNY17-1

Commit message: Re-generated Henning's board using a different terminal block.
Parts:
- P2: footprint Terminal_Blocks:TerminalBlock_WAGO-236_2Stift_RM5mm_2pol -> Terminal_Blocks:TerminalBlock_Pheonix_MPT-2.54mm_2pol
- moved P2 6.67 mm to (71.2, 45.8)
Routing:
- net EBUS1: track 25.3 -> 29.8 mm
- net EBUS2: track 17.4 -> 21.1 mm
