File: Tony_Groeger/Groeger.sch (KiCad schematic (older format))
At the start: 14 parts, among them P1 EBUS, P2 RS232, Q1 PN2222A, U1 7805, U2 4011

Commit message: PCB generated.
Parts:
- C1, C2: footprint (none) -> Capacitors_ThroughHole:C_Disc_D3_P2.5
- D1, D2, D3: footprint (none) -> Diodes_ThroughHole:Diode_DO-41_SOD81_Horizontal_RM10
- D4: footprint (none) -> LEDs:LED-5MM
- P1: footprint (none) -> Terminal_Blocks:TerminalBlock_Pheonix_PT-3.5mm_2pol
- P2: footprint (none) -> Pin_Headers:Pin_Header_Straight_1x02
- Q1, U1: footprint (none) -> TO_SOT_Packages_THT:TO-92_Molded_Wide
- R1, R2: footprint (none) -> Resistors_ThroughHole:Resistor_Horizontal_RM10mm
- RV1: footprint (none) -> Potentiometers:Potentiometer_Bourns_3296W_3-8Zoll_Inline_ScrewUp
- U2: footprint (none) -> Housings_DIP:DIP-14_W7.62mm
Connections:
- wire segments 40 -> 41
Changed lines of the file:
@@
 F 0 "P1" H 1850 1300 50  0000 C CNN
 F 1 "EBUS" V 1950 1150 50  0000 C CNN
-F 2 "" H 1850 1150 50  0000 C CNN
+F 2 "Terminal_Blocks:TerminalBlock_Pheonix_PT-3.5mm_2pol" H 1850 1150 50  0001 C CNN
 F 3 "" H 1850 1150 50  0000 C CNN
 	1    1850 1150
@@
 F 0 "U1" H 4350 1804 50  0000 C CNN
 F 1 "7805" H 4200 2200 50  0000 C CNN
-F 2 "" H 4200 2000 50  0000 C CNN
+F 2 "TO_SOT_Packages_THT:TO-92_Molded_Wide" H 4200 2000 50  0001 C CNN
 F 3 "" H 4200 2000 50  0000 C CNN
 	1    4200 2000
@@
 F 0 "C1" H 3625 2200 50  0000 L CNN
 F 1 "100pF" H 3625 2000 50  0000 L CNN
-F 2 "" H 3638 1950 50  0000 C CNN
+F 2 "Capacitors_ThroughHole:C_Disc_D3_P2.5" H 3638 1950 50  0001 C CNN
 F 3 "" H 3600 2100 50  0000 C CNN
 	1    3600 2100
@@
 F 0 "C2" H 4825 2200 50  0000 L CNN
 F 1 "100pF" H 4825 2000 50  0000 L CNN
-F 2 "" H 4838 1950 50  0000 C CNN
+F 2 "Capacitors_ThroughHole:C_Disc_D3_P2.5" H 4838 1950 50  0001 C CNN
 F 3 "" H 4800 2100 50  0000 C CNN
 	1    4800 2100
@@
 F 0 "D4" H 5200 2250 50  0000 C CNN
 F 1 "LED" H 5200 2050 50  0000 C CNN
-F 2 "" H 5200 2150 50  0000 C CNN
+F 2 "LEDs:LED-5MM" H 5200 2150 50  0001 C CNN
 F 3 "" H 5200 2150 50  0000 C CNN
 	1    5200 2150
@@
 F 0 "R2" V 5280 2600 50  0000 C CNN
 F 1 "470" V 5200 2600 50  0000 C CNN
-F 2 "" V 5130 2600 50  0000 C CNN
+F 2 "Resistors_ThroughHole:Resistor_Horizontal_RM10mm" V 5130 2600 50  0001 C CNN
 F 3 "" H 5200 2600 50  0000 C CNN
 	1    5200 2600
@@
 F 0 "D2" H 2600 2800 50  0000 C CNN
 F 1 "1N4148" H 2600 2600 50  0000 C CNN
-F 2 "" H 2600 2700 50  0000 C CNN
+F 2 "Diodes_ThroughHole:Diode_DO-41_SOD81_Horizontal_RM10" H 2600 2700 50  0001 C CNN
 F 3 "" H 2600 2700 50  0000 C CNN
 	1    2600 2700
@@
 F 0 "D1" H 2600 2350 50  0000 C CNN
 F 1 "1N4148" H 2600 2150 50  0000 C CNN
-F 2 "" H 2600 2250 50  0000 C CNN
+F 2 "Diodes_ThroughHole:Diode_DO-41_SOD81_Horizontal_RM10" H 2600 2250 50  0001 C CNN
 F 3 "" H 2600 2250 50  0000 C CNN
 	1    2600 2250
@@
 F 0 "D3" H 2600 3300 50  0000 C CNN
 F 1 "7.5V/1.3W" H 2600 3100 50  0000 C CNN
-F 2 "" H 2600 3200 50  0000 C CNN
+F 2 "Diodes_ThroughHole:Diode_DO-41_SOD81_Horizontal_RM10" H 2600 3200 50  0001 C CNN
 F 3 "" H 2600 3200 50  0000 C CNN
 	1    2600 3200
@@
 F 0 "R1" V 2030 3800 50  0000 C CNN
 F 1 "8k" V 1950 3800 50  0000 C CNN
-F 2 "" V 1880 3800 50  0000 C CNN
+F 2 "Resistors_ThroughHole:Resistor_Horizontal_RM10mm" V 1880 3800 50  0001 C CNN
 F 3 "" H 1950 3800 50  0000 C CNN
 	1    1950 3800
@@
 F 0 "Q1" H 2700 3875 50  0000 L CNN
 F 1 "PN2222A" H 2700 3800 50  0000 L CNN
-F 2 "" H 2700 3725 50  0000 L CIN
+F 2 "TO_SOT_Packages_THT:TO-92_Molded_Wide" H 2700 3725 50  0001 L CIN
 F 3 "" H 2500 3800 50  0000 L CNN
 	1    2500 3800
@@
 F 0 "U2" H 6150 3800 50  0000 C CNN
 F 1 "4011" H 6150 3700 50  0000 C CNN
-F 2 "" H 6150 3750 60  0000 C CNN
+F 2 "Housings_DIP:DIP-14_W7.62mm" H 6150 3750 60  0001 C CNN
 F 3 "" H 6150 3750 60  0000 C CNN
 	1    6150 3750
@@
 F 0 "U2" H 7800 3700 50  0000 C CNN
 F 1 "4011" H 7800 3600 50  0000 C CNN
-F 2 "" H 7800 3650 60  0000 C CNN
+F 2 "Housings_DIP:DIP-14_W7.62mm" H 7800 3650 60  0001 C CNN
 F 3 "" H 7800 3650 60  0000 C CNN
 	3    7800 3650
@@
 F 0 "U2" H 7750 4600 50  0000 C CNN
 F 1 "4011" H 7750 4500 50  0000 C CNN
-F 2 "" H 7750 4550 60  0000 C CNN
+F 2 "Housings_DIP:DIP-14_W7.62mm" H 7750 4550 60  0001 C CNN
 F 3 "" H 7750 4550 60  0000 C CNN
 	2    7750 4550
@@
 F 0 "P2" H 9600 2300 50  0000 C CNN
 F 1 "RS232" V 9700 2150 50  0000 C CNN
-F 2 "" H 9600 2150 50  0000 C CNN
+F 2 "Pin_Headers:Pin_Header_Straight_1x02" H 9600 2150 50  0001 C CNN
 F 3 "" H 9600 2150 50  0000 C CNN
 	1    9600 2150
@@
 EBUS+
 $Comp
-L GND #PWR1
+L GND #PWR01
 U 1 1 57E4FA3D
 P 2600 1500
-F 0 "#PWR1" H 2600 1250 50  0001 C CNN
+F 0 "#PWR01" H 2600 1250 50  0001 C CNN
 F 1 "GND" H 2600 1350 50  0000 C CNN
 F 2 "" H 2600 1500 50  0000 C CNN
@@
 	2600 1700 2600 1500
 $Comp
-L GND #PWR2
+L GND #PWR02
 U 1 1 57E4FFD4
 P 2600 4150
-F 0 "#PWR2" H 2600 3900 50  0001 C CNN
+F 0 "#PWR02" H 2600 3900 50  0001 C CNN
 F 1 "GND" H 2600 4000 50  0000 C CNN
 F 2 "" H 2600 4150 50  0000 C CNN
@@
 F 0 "RV1" H 3300 3770 50  0000 C CNN
 F 1 "10k" H 3300 3850 50  0000 C CNN
-F 2 "" H 3300 3850 50  0000 C CNN
+F 2 "Potentiometers:Potentiometer_Bourns_3296W_3-8Zoll_Inline_ScrewUp" H 3300 3850 50  0001 C CNN
 F 3 "" H 3300 3850 50  0000 C CNN
 	1    3300 3850
@@
 Connection ~ 3300 1950
 $Comp
-L GND #PWR3
+L GND #PWR03
 U 1 1 57E4F99C
 P 4200 3050
-F 0 "#PWR3" H 4200 2800 50  0001 C CNN
+F 0 "#PWR03" H 4200 2800 50  0001 C CNN
 F 1 "GND" H 4200 2900 50  0000 C CNN
 F 2 "" H 4200 3050 50  0000 C CNN
@@
 Connection ~ 5550 1950
 $Comp
-L GND #PWR4
+L GND #PWR04
 U 1 1 57E4FF6B
 P 5950 4100
-F 0 "#PWR4" H 5950 3850 50  0001 C CNN
+F 0 "#PWR04" H 5950 3850 50  0001 C CNN
 F 1 "GND" H 5950 3950 50  0000 C CNN
 F 2 "" H 5950 4100 50  0000 C CNN
@@
 	6750 3750 7200 3750
 Wire Wire Line
-	7150 1950 7150 3500
+	7150 1950 7150 3550
 Connection ~ 5950 1950
 Wire Wire Line
@@
 Wire Wire Line
 	9400 2200 8800 2200
+Wire Wire Line
+	7150 3550 7200 3550
 $EndSCHEMATC

Commit message: Changed Groeger's PCB terminal block component to something we have on hand.
Parts:
- P1: footprint Terminal_Blocks:TerminalBlock_Pheonix_PT-3.5mm_2pol -> Terminal_Blocks:TerminalBlock_Pheonix_MKDS1.5-2pol
Changed lines of the file:
@@
 F 0 "P1" H 1850 1300 50  0000 C CNN
 F 1 "EBUS" V 1950 1150 50  0000 C CNN
-F 2 "Terminal_Blocks:TerminalBlock_Pheonix_PT-3.5mm_2pol" H 1850 1150 50  0001 C CNN
+F 2 "Terminal_Blocks:TerminalBlock_Pheonix_MKDS1.5-2pol" H 1850 1150 50  0001 C CNN
 F 3 "" H 1850 1150 50  0000 C CNN
 	1    1850 1150
